File: PCB/kicad/Audio_Devboard.kicad_pcb (KiCad board)
At the start: 4 copper layers, 56 x 37 mm, 85 parts, among them J1 Black headphone jack, J2 Black headphone jack, J4 Conn_01x08, SW1 SW_Push, SW2 SW_Push, SW3 SW_Push, SW4 SW_Push, SW5 SW_Push, SW6 SW_Push, U1 VS1053B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

Commit message: Rev 1.0.0
Parts:
- added R26: 20R, Resistor_SMD:R_0402_1005Metric, F.Cu at (115.2, 107.1)
- added R27: 20R, Resistor_SMD:R_0402_1005Metric, F.Cu at (120.2, 107.1)
- C10, C15, C5: value 10Uf 6V3 -> 10uF 6V3
- C14, C9: value LC -> 18pF
- Y1: value Crystal_GND24 -> SX2B12.288F1210F30
- moved C12 1.01 mm to (121.2, 107.1)
- moved SW3 0.20 mm to (99.5, 103.2)
- moved SW4 0.20 mm to (110.3, 103.2)
- moved SW5 0.20 mm to (121.2, 103.2)
- moved SW6 0.20 mm to (132.0, 103.2)
- moved C11 0.16 mm to (116.2, 107.1)
- moved C13 0.16 mm to (118.2, 107.1)
- moved C15 0.16 mm to (119.2, 107.1)
- moved C16 0.16 mm to (117.2, 107.1)
Connections:
- J1 pad 2: /RIGHT -> Net-(J1-R)
- J1 pad 4: /LEFT -> Net-(J1-L)
- R4 pad 2: /RIGHT -> Net-(J1-R)
- R5 pad 2: /LEFT -> Net-(J1-L)
Routing:
- net Net-(J1-R): track 0.00 -> 41.1 mm, vias 0 -> 1
- net /RIGHT: track 40.4 -> 1.88 mm, vias 1 -> 0
- net Net-(J1-L): track 0.00 -> 22.2 mm, vias 0 -> 1
- net /LEFT: track 20.4 -> 2.13 mm, vias 1 -> 0
- net +3V3: track 168.6 -> 156.2 mm
- net /PA2: track 37.5 -> 39.8 mm
- net /PA1: track 38.1 -> 39.8 mm
- net /VS_GP4: track 22.0 -> 23.2 mm
- net /VS_GP1: track 34.2 -> 35.3 mm
- net GND: track 40.8 -> 41.7 mm
