File: PCB/kicad/Audio_Devboard.kicad_sch (KiCad schematic)
At the start: 85 parts, among them J1 Black headphone jack, J2 Black headphone jack, J4 Conn_01x08, SW1 SW_Push, SW2 SW_Push, SW3 SW_Push, SW4 SW_Push, SW5 SW_Push, SW6 SW_Push, U1 VS1053B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

Commit message: Rev 1.0.0
Parts:
- added R26, R27: 20R, Resistor_SMD:R_0402_1005Metric, symbol Device:R
- C1, C11, C12, C13, C2, C24, C25, C26, C3, C31, C4, C6, C7, C8: LCSC Part (none) -> C1525
- C10, C15, C5: value 10Uf 6V3 -> 10uF 6V3; symbol Device:C_Polarized -> Device:C; LCSC Part (none) -> C315248
- C14, C9: value LC -> 18pF; LCSC Part (none) -> C106202
- C16, C22, C23, C27, C28, C29, C30: LCSC Part (none) -> C14445
- C17: LCSC Part (none) -> C368599
- C18, C19: LCSC Part (none) -> C15195
- C20, C21: LCSC Part (none) -> C3855387
- D1, D2, D3, D4, D5, D6: LCSC Part (none) -> C364553
- J4: LCSC Part (none) -> C6332201
- R1: LCSC Part (none) -> C138033
- R10, R11, R12, R19, R2, R20, R21, R9: LCSC Part (none) -> C166559
- R13, R14: LCSC Part (none) -> C25905
- R15, R16, R17, R18, R22, R24, R25: LCSC Part (none) -> 0402WGF1002TCE C25744 Hot
- R23, R6: LCSC Part (none) -> C25741
- R3: LCSC Part (none) -> C25077
- R4, R5: LCSC Part (none) -> C25089
- R7, R8: LCSC Part (none) -> C25117
- SW1, SW2, SW3, SW4, SW5, SW6: LCSC Part (none) -> C393938
- TP1, TP2, TP3: now left out of the parts list
- Y1: value Crystal_GND24 -> SX2B12.288F1210F30; LCSC Part (none) -> C49253544
Connections:
- net LEFT: now also R26.1; no longer J1.4 (L), R5.2
- net RIGHT: now also R27.1; no longer J1.2 (R), R4.2
- new net: J1.4 (L), R26.2, R5.2
- new net: J1.2 (R), R27.2, R4.2
Other:
- moved on the sheet: C17, C18, C19, J1, R3, R4, R5
